Commit message: added IMU sensor plugin and finalized robot model

File: robot_description/urdf/mobile_robot.urdf (robot description, URDF)
Before this commit: robot mobile_robot, 4 links, 3 joints
Links:
- link imu_link: mass None -> 0.1
- link left_wheel: mass None -> 1.0; geometry collision cylinder length=0.02 radius=0.05; visual cylinder length=0.02 radius=0.05
- link right_wheel: mass None -> 1.0; geometry collision cylinder length=0.02 radius=0.05; visual cylinder length=0.02 radius=0.05
