Commit message: configuration for ROS2 Humble and environment setup

File: mar_imu/robot_description/urdf/mobile_robot.urdf (robot description, URDF)
Before this commit: robot mobile_robot, 4 links, 3 joints
Links:
- link base_link: mass 5.0 -> 2.0
- link left_wheel: mass 1.0 -> 0.5
- link right_wheel: mass 1.0 -> 0.5
Joints:
- joint left_wheel_joint: origin xyz=0 0.15 -0.05 rpy=0 1.57 0 -> xyz=0 0.15 -0.03 rpy=0 1.57 0
- joint right_wheel_joint: origin xyz=0 -0.15 -0.05 rpy=0 1.57 0 -> xyz=0 -0.15 -0.03 rpy=0 1.57 0

Commit message: fix: teleporting issues and the teleop issues,please verify

File: mar_imu/robot_description/urdf/mobile_robot.urdf (robot description, URDF)
Before this commit: robot mobile_robot, 4 links, 3 joints
Joints:
- joint left_wheel_joint: origin xyz=0 0.15 -0.05 rpy=0 1.57 0 -> xyz=0 0.15 -0.05 rpy=1.5708 0 0
- joint right_wheel_joint: origin xyz=0 -0.15 -0.05 rpy=0 1.57 0 -> xyz=0 -0.15 -0.05 rpy=1.5708 0 0
